File: hardware/rev_a/thread_dongle.sch (EAGLE design)
At the start: 24 parts, among them J1 USB-A-MALE-PLUG, J2 TC2030-JLINK-NL, U1 KW21Z, U2 ESDR0502N, U3 CP2102N-20, X1 FA-128, X2 FA-135

Commit message: Nothing to do and no errors
Parts:
- added C6, C7: 12pF, passives:CAPACITOR0402_CAP
Connections:
- removed net N$11: U1.EXTAL, X1.2
- removed net N$14: U1.PTB17/XTAL32K, X2.1
- removed net N$15: U1.PTB16/EXTAL32K, X2.2
- new net N$1: C6.1, U1.PTB16/EXTAL32K, X2.2
- new net N$2: C7.1, U1.PTB17/XTAL32K, X2.1
- new net N$3: U1.XTAL, X1.2
- net GND: now also C6.2, C7.2
- net N$12: now also U1.EXTAL; no longer U1.XTAL
Other:
- note added: "C10, C11, C12 place close to pin 20, 44, 28"
- note added: "C13, C14 place close to pins 36, 35"
- moved on the sheet: X1, X2
Changed lines of the file:
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@@
 <part name="SJ1" library="headers" deviceset="SOLDERJUMPER" device="NC"/>
 <part name="SJ2" library="headers" deviceset="SOLDERJUMPER" device="NC"/>
+<part name="C6" library="passives" deviceset="CAPACITOR" device="0402_CAP" value="12pF">
+<attribute name="DIGIKEY" value="490-5924-1-ND"/>
+</part>
+<part name="C7" library="passives" deviceset="CAPACITOR" device="0402_CAP" value="12pF">
+<attribute name="DIGIKEY" value="490-5924-1-ND"/>
+</part>
+<part name="GND1" library="supply1" library_urn="urn:adsk.eagle:library:371" deviceset="GND" device=""/>
 </parts>
 <sheets>
@@
 <plain>
 <text x="88.9" y="73.66" size="1.016" layer="98" align="bottom-center">FLOWCONTROL ENABLE</text>
+<text x="152.4" y="177.8" size="1.016" layer="98">C10, C11, C12 place close to pin 20, 44, 28</text>
+<text x="152.4" y="154.94" size="1.016" layer="98">C13, C14 place close to pins 36, 35</text>
 </plain>
 <instances>
@@
 <instance part="P+5" gate="VCC" x="147.32" y="180.34"/>
 <instance part="GND8" gate="1" x="147.32" y="144.78"/>
-<instance part="X1" gate="G$1" x="152.4" y="129.54">
-<attribute name="DIGIKEY" x="152.4" y="129.54" size="1.778" layer="96" display="off"/>
-</instance>
-<instance part="X2" gate="G$1" x="165.1" y="139.7">
-<attribute name="DIGIKEY" x="165.1" y="139.7" size="1.778" layer="96" display="off"/>
-</instance>
-<instance part="GND11" gate="1" x="152.4" y="116.84"/>
+<instance part="X1" gate="G$1" x="157.48" y="116.84">
+<attribute name="DIGIKEY" x="157.48" y="116.84" size="1.778" layer="96" display="off"/>
+</instance>
+<instance part="X2" gate="G$1" x="157.48" y="134.62" rot="MR0">
+<attribute name="DIGIKEY" x="157.48" y="134.62" size="1.778" layer="96" rot="MR0" display="off"/>
+</instance>
+<instance part="GND11" gate="1" x="157.48" y="104.14"/>
 <instance part="L1" gate="G$1" x="231.14" y="106.68" rot="R270">
 <attribute name="DIGIKEY" x="231.14" y="106.68" size="1.778" layer="96" rot="R270" display="off"/>
@@
 <attribute name="NAME" x="86.36" y="63.5" size="1.778" layer="95"/>
 </instance>
+<instance part="C6" gate="G$1" x="147.32" y="132.08">
+<attribute name="DIGIKEY" x="147.32" y="132.08" size="1.778" layer="96" display="off"/>
+</instance>
+<instance part="C7" gate="G$1" x="165.1" y="132.08">
+<attribute name="DIGIKEY" x="165.1" y="132.08" size="1.778" layer="96" display="off"/>
+</instance>
+<instance part="GND1" gate="1" x="144.78" y="121.92"/>
 </instances>
 <busses>
@@
 <segment>
 <pinref part="X1" gate="G$1" pin="GND"/>
-<wire x1="152.4" y1="124.46" x2="152.4" y2="119.38" width="0.1524" layer="91"/>
+<wire x1="157.48" y1="111.76" x2="157.48" y2="106.68" width="0.1524" layer="91"/>
 <pinref part="GND11" gate="1" pin="GND"/>
 </segment>
@@
 <pinref part="GND13" gate="1" pin="GND"/>
 <wire x1="220.98" y1="99.06" x2="220.98" y2="96.52" width="0.1524" layer="91"/>
+</segment>
+<segment>
+<pinref part="C7" gate="G$1" pin="2"/>
+<pinref part="C6" gate="G$1" pin="2"/>
+<wire x1="165.1" y1="127" x2="147.32" y2="127" width="0.1524" layer="91"/>
+<junction x="147.32" y="127"/>
+<pinref part="GND1" gate="1" pin="GND"/>
+<wire x1="144.78" y1="124.46" x2="144.78" y2="127" width="0.1524" layer="91"/>
+<wire x1="144.78" y1="127" x2="147.32" y2="127" width="0.1524" layer="91"/>
 </segment>
 </net>
@@
 </segment>
 </net>
-<net name="N$11" class="0">
-<segment>
-<pinref part="X1" gate="G$1" pin="2"/>
-<wire x1="157.48" y1="129.54" x2="160.02" y2="129.54" width="0.1524" layer="91"/>
-<wire x1="160.02" y1="129.54" x2="160.02" y2="127" width="0.1524" layer="91"/>
+<net name="N$12" class="0">
+<segment>
+<pinref part="X1" gate="G$1" pin="1"/>
+<wire x1="149.86" y1="116.84" x2="152.4" y2="116.84" width="0.1524" layer="91"/>
+<wire x1="149.86" y1="116.84" x2="149.86" y2="121.92" width="0.1524" layer="91"/>
+<wire x1="149.86" y1="121.92" x2="175.26" y2="121.92" width="0.1524" layer="91"/>
+<wire x1="175.26" y1="121.92" x2="175.26" y2="127" width="0.1524" layer="91"/>
 <pinref part="U1" gate="G$1" pin="EXTAL"/>
-<wire x1="160.02" y1="127" x2="180.34" y2="127" width="0.1524" layer="91"/>
-</segment>
-</net>
-<net name="N$12" class="0">
-<segment>
-<pinref part="U1" gate="G$1" pin="XTAL"/>
-<wire x1="180.34" y1="124.46" x2="160.02" y2="124.46" width="0.1524" layer="91"/>
-<wire x1="160.02" y1="124.46" x2="160.02" y2="121.92" width="0.1524" layer="91"/>
-<wire x1="160.02" y1="121.92" x2="144.78" y2="121.92" width="0.1524" layer="91"/>
-<wire x1="144.78" y1="121.92" x2="144.78" y2="129.54" width="0.1524" layer="91"/>
-<pinref part="X1" gate="G$1" pin="1"/>
-<wire x1="144.78" y1="129.54" x2="147.32" y2="129.54" width="0.1524" layer="91"/>
-</segment>
-</net>
-<net name="N$14" class="0">
-<segment>
-<pinref part="U1" gate="G$1" pin="PTB17/XTAL32K"/>
-<wire x1="157.48" y1="132.08" x2="180.34" y2="132.08" width="0.1524" layer="91"/>
-<pinref part="X2" gate="G$1" pin="1"/>
-<wire x1="160.02" y1="139.7" x2="157.48" y2="139.7" width="0.1524" layer="91"/>
-<wire x1="157.48" y1="139.7" x2="157.48" y2="132.08" width="0.1524" layer="91"/>
-</segment>
-</net>
-<net name="N$15" class="0">
-<segment>
-<pinref part="U1" gate="G$1" pin="PTB16/EXTAL32K"/>
-<wire x1="180.34" y1="134.62" x2="172.72" y2="134.62" width="0.1524" layer="91"/>
-<wire x1="172.72" y1="134.62" x2="172.72" y2="139.7" width="0.1524" layer="91"/>
-<pinref part="X2" gate="G$1" pin="2"/>
-<wire x1="172.72" y1="139.7" x2="170.18" y2="139.7" width="0.1524" layer="91"/>
+<wire x1="175.26" y1="127" x2="180.34" y2="127" width="0.1524" layer="91"/>
 </segment>
 </net>
@@
 </segment>
 </net>
+<net name="N$1" class="0">
+<segment>
+<pinref part="C6" gate="G$1" pin="1"/>
+<pinref part="U1" gate="G$1" pin="PTB16/EXTAL32K"/>
+<wire x1="180.34" y1="134.62" x2="177.8" y2="134.62" width="0.1524" layer="91"/>
+<wire x1="177.8" y1="134.62" x2="177.8" y2="139.7" width="0.1524" layer="91"/>
+<wire x1="177.8" y1="139.7" x2="147.32" y2="139.7" width="0.1524" layer="91"/>
+<wire x1="147.32" y1="139.7" x2="147.32" y2="134.62" width="0.1524" layer="91"/>
+<pinref part="X2" gate="G$1" pin="2"/>
+<wire x1="152.4" y1="134.62" x2="147.32" y2="134.62" width="0.1524" layer="91"/>
+<junction x="147.32" y="134.62"/>
+</segment>
+</net>
+<net name="N$2" class="0">
+<segment>
+<pinref part="C7" gate="G$1" pin="1"/>
+<pinref part="U1" gate="G$1" pin="PTB17/XTAL32K"/>
+<wire x1="180.34" y1="132.08" x2="175.26" y2="132.08" width="0.1524" layer="91"/>
+<wire x1="175.26" y1="132.08" x2="175.26" y2="134.62" width="0.1524" layer="91"/>
+<wire x1="175.26" y1="134.62" x2="165.1" y2="134.62" width="0.1524" layer="91"/>
+<pinref part="X2" gate="G$1" pin="1"/>
+<wire x1="162.56" y1="134.62" x2="165.1" y2="134.62" width="0.1524" layer="91"/>
+<junction x="165.1" y="134.62"/>
+</segment>
+</net>
+<net name="N$3" class="0">
+<segment>
+<pinref part="U1" gate="G$1" pin="XTAL"/>
+<wire x1="180.34" y1="124.46" x2="177.8" y2="124.46" width="0.1524" layer="91"/>
+<wire x1="177.8" y1="124.46" x2="177.8" y2="116.84" width="0.1524" layer="91"/>
+<pinref part="X1" gate="G$1" pin="2"/>
+<wire x1="177.8" y1="116.84" x2="162.56" y2="116.84" width="0.1524" layer="91"/>
+</segment>
+</net>

Commit message: Fix up silkscreen
Parts:
- C1, C10, C11, C12, C3: DIGIKEY (none) -> 587-1227-1-ND; MPN (none) -> LMK105BJ104KV-F
- C13, C14, C6, C7: MPN (none) -> GRM1555C1H120JA01D
- C2: DIGIKEY (none) -> 490-5915-1-ND; MPN (none) -> GRM155R60J475ME47D
- C4: DIGIKEY (none) -> 490-10018-1-ND; MPN (none) -> GRM155R61E105MA12D
- C5: MPN (none) -> GRM1555C1HR70BA01D
- D1: DIGIKEY (none) -> 160-1837-6-ND; MPN (none) -> LTST-C194TBKT
- L1: MPN (none) -> LQG15HS5N1S02D
- R1: DIGIKEY (none) -> 311-10KJRCT-ND; MPN (none) -> RC0402JR-0710KL
- R8: DIGIKEY (none) -> 311-1.0KJRCT-ND; MPN (none) -> RC0402JR-071KL
- X1: MPN (none) -> FA-128 32.0000MF20X-K5
- X2: MPN (none) -> FC-135 32.7680KA-AG3
Other:
- moved on the sheet: D1

Commit message: ship it
Parts:
- removed C13, C14: 12pF, passives:CAPACITOR0402_CAP
- removed R8: 1k, passives:RESISTOR0402_RES
- added C8, C9: 0.1uF, passives:CAPACITOR0402_CAP
- added R2: 10k, passives:RESISTOR0402_RES
- C1: value 0.1uF -> 0.7pF; DIGIKEY 587-1227-1-ND -> 490-6267-1-ND; MPN LMK105BJ104KV-F -> GRM1555C1HR70BA01D
- C11: value 0.1uF -> 1.0uF; DIGIKEY 587-1227-1-ND -> 490-10018-1-ND; MPN LMK105BJ104KV-F -> GRM155R61E105MA12D
- C12: value 0.1uF -> 4.7uF; DIGIKEY 587-1227-1-ND -> 490-5915-1-ND; MPN LMK105BJ104KV-F -> GRM155R60J475ME47D
- C2: value 4.7uF -> 12pF; DIGIKEY 490-5915-1-ND -> 490-5924-1-ND; MPN GRM155R60J475ME47D -> GRM1555C1H120JA01D
- C3: value 0.1uF -> 12pF; DIGIKEY 587-1227-1-ND -> 490-5924-1-ND; MPN LMK105BJ104KV-F -> GRM1555C1H120JA01D
- C4: value 1.0uF -> 12pF; DIGIKEY 490-10018-1-ND -> 490-5924-1-ND; MPN GRM155R61E105MA12D -> GRM1555C1H120JA01D
- C5: value 0.7pF -> 12pF; DIGIKEY 490-6267-1-ND -> 490-5924-1-ND; MPN GRM1555C1HR70BA01D -> GRM1555C1H120JA01D
- C6, C7: value 12pF -> 0.1uF; DIGIKEY 490-5924-1-ND -> 587-1227-1-ND; MPN GRM1555C1H120JA01D -> LMK105BJ104KV-F
- J1: value USB-A-MALE-PLUG -> TC2030-JLINK-NL; device connector:USB-A-MALE-PLUG -> connector:TC2030-JLINK-NL
- J2: value TC2030-JLINK-NL -> USB-A-MALE-PLUG; device connector:TC2030-JLINK-NL -> connector:USB-A-MALE-PLUG
- R1: value 10k -> 1k; DIGIKEY 311-10KJRCT-ND -> 311-1.0KJRCT-ND; MPN RC0402JR-0710KL -> RC0402JR-071KL
- U1: value KW21Z -> CP2102N-20; device chips:KW21Z -> chips:CP2102N-20
- U3: value CP2102N-20 -> KW21Z; device chips:CP2102N-20 -> chips:KW21Z
Connections:
- removed net SWCLK: J2.SWDCLK, U1.SWD_DIO
- new net SWDCLK: J1.SWDCLK, U3.SWD_CLK
- net !RESET: now also J1.!RESET, R2.1, U1.!RST, U3.RESET; no longer J2.!RESET, R1.1, U1.RESET, U3.!RST
- net 5V: now also C11.1, C7.1, J2.+5V, U1.VBUS, U1.VREGIN; no longer C3.1, C4.1, J1.+5V, U3.VBUS, U3.VREGIN
- net CP_CTS: now also U1.CTS; no longer U3.CTS
- net CP_RTS: now also U1.RTS; no longer U3.RTS
- net D+: now also J2.D+, U1.D+; no longer J1.D+, U3.D+
- net D-: now also J2.D-, U1.D-; no longer J1.D-, U3.D-
- net GND: now also C8.2, C9.2, U3.PSWITCH; no longer C13.2, C14.2, U1.PSWITCH
- net KW21Z_CTS: now also U3.PTC4; no longer U1.PTC4
- net KW21Z_RTS: now also U3.PTC5; no longer U1.PTC5
- net KW21Z_RX: now also U1.TXD, U3.PTC2; no longer U1.PTC2, U3.TXD
- net KW21Z_TX: now also U1.RXD, U3.PTC3; no longer U1.PTC3, U3.RXD
- net N$1: now also C4.1, U3.PTB16/EXTAL32K; no longer C6.1, U1.PTB16/EXTAL32K
- net N$12: now also U3.EXTAL; no longer U1.EXTAL
- net N$13: now also C1.1, U3.ANT; no longer C5.1, U1.ANT
- net N$2: now also C5.1, U3.PTB17/XTAL32K; no longer C7.1, U1.PTB17/XTAL32K
- net N$3: now also U3.XTAL; no longer U1.XTAL
- net N$7: now also R1.2; no longer R8.2
- net N$8: now also R1.1, U3.PTB0; no longer R8.1, U1.PTB0
- net SWDIO: now also J1.SWDIO, U3.SWD_DIO; no longer J2.SWDIO, U1.SWD_CLK
- net VCC: now also C3.1, C6.1, C8.1, C9.1, J1.VCC, R2.2, U3.DCDC_CFG, U3.VDDA, U3.VDD_1P5/PMC, U3.VDD_1P8_OUT, U3.VDD_RF, U3.VREFH; no longer C1.1, C11.1, C13.1, C14.1, J2.VCC, R1.2, U1.DCDC_CFG, U1.VDDA, U1.VDD_1P5/PMC, U1.VDD_1P8_OUT, U1.VDD_RF, U1.VREFH
Other:
- moved on the sheet: C1, C10, C11, C12, C2, C3, C4, C5, C6, C7, R1
